Commit message: feat: Update sensor to simulated Kinect camera for RTAB-Map

File: my_robot/urdf/my_robot.xacro (robot description, xacro)
@@ -193,3 +193,10 @@
         <axis xyz="0 1 0" />
   </joint>
+ <joint name="camera_optical_joint" type="fixed">
+    <origin xyz="0 0 0" rpy="-1.5707 0 -1.5707"/>
+    <parent link="camera"/>
+    <child link="camera_link_optical"/>
+  </joint>
+  <link name="camera_link_optical">
+  </link>
 </robot>

Commit message: refactor: Modify the robot xacro file

File: my_robot/urdf/my_robot.xacro (robot description, xacro)
@@ -188,15 +188,15 @@
   </link>
   <joint name="hokuyo" type="fixed">
-	<origin xyz="0.25 0 0.15" rpy="0 0 0" />
+        <origin xyz="0.25 0 0.15" rpy="0 0 0" />
 	<child link="hokuyo" />
 	<parent link="chassis" />
         <axis xyz="0 1 0" />
   </joint>
- <joint name="camera_optical_joint" type="fixed">
-    <origin xyz="0 0 0" rpy="-1.5707 0 -1.5707"/>
-    <parent link="camera"/>
-    <child link="camera_link_optical"/>
-  </joint>
   <link name="camera_link_optical">
   </link>
+  <joint name="camera_optical_joint" type="fixed">
+     <origin xyz="0 0 0" rpy="-1.5707 0 -1.5707"/>
+     <parent link="camera"/>
+     <child link="camera_link_optical"/>
+  </joint>
 </robot>
